Commit message: final version with real sensor

File: model/ft_sensor.gazebo.xacro (robot description, xacro)
@@ -17,5 +17,5 @@
 <!--       <provideFeedback>true</provideFeedback> -->
     </gazebo>
-    <gazebo reference="${name}_imu_measure">
+     <gazebo reference="${name}_imu_measure">
       <material>Gazebo/Blue</material>
      <sensor name='imu_sensor' type='imu'>
@@ -30,5 +30,4 @@
     <bodyName>${name}_imu_measure</bodyName>
     <updateRateHZ>1000.0</updateRateHZ>
-    <!-- <gaussianNoise>0.0</gaussianNoise> -->
     <gaussianNoise>0.003</gaussianNoise>
     <xyzOffset>0.0 0.0 0.0</xyzOffset>
@@ -49,5 +48,5 @@
 		</gazebo>
     <!-- The ft_sensor plugin  -->
-    <gazebo>
+     <gazebo>
         <plugin name="ft_sensor" filename="libgazebo_ros_ft_sensor.so">
         <updateRate>1000.0</updateRate>
@@ -57,5 +56,5 @@
           <type>gaussian</type>
           <mean>0.0</mean>
-          <stddev>0.003</stddev> <!-- change this to simulate noise  0.003-->
+          <stddev>0.003</stddev>
         </noise>
         </plugin>

File: model/ft_sensor.trasmission.xacro (robot description, xacro)
@@ -6,8 +6,9 @@
           <robotNamespace>/${name}/</robotNamespace>
        </plugin>
+ <!--
        	 <ros>
            <plugin name="${name}_contact_point_estimato" filename="libcontact_point_estimator.so">
 	   </plugin>
-	 </ros>
+	 </ros>-->
 	</xacro:macro>
 </robot>

File: model/ft_sensor_gamma.urdf.xacro (robot description, xacro)
@@ -32,5 +32,6 @@
 			<child link="${name}_imu_measure"/>
 			<axis xyz="0 0 1" />
-			<origin rpy="1.57 -1.57 -1.57" xyz="-0.0378 0 0.01665"/>
+			<!--origin rpy="1.57 -1.57 -1.57" xyz="-0.0378 0 0.01665"/-->
+			<origin rpy="-1.57 -1.57 -1.57" xyz=" -0.025 0.025 0.14"/>
 <!-- 			<dynamics damping="10.0" friction="10.0"/>
 			 <limit lower="0" upper="0" effort="0" velocity="0"/>
